File: circuit/1x9/1x9.sch (KiCad schematic (older format))
At the start: 22 parts

Commit message: v1.1
Parts:
- removed JIN3, JOUT4: Conn_01x08_Shielded, Connector_JST:JST_SUR_BM08B-SURS-TF_1x08-1MP_P0.80mm_Vertical, symbol Connector_Generic:Conn_01x08
- added JIN1, JOUT1: Conn_01x05, library:thick_header_01x05_3.3mm, symbol Connector_Generic:Conn_01x05
- JIN2, JOUT3: value Conn_01x08_Shielded -> Conn_01x05; footprint Connector_JST:JST_SUR_BM08B-SURS-TF_1x08-1MP_P0.80mm_Vertical -> library:thick_header_01x05_3.3mm; symbol Connector_Generic:Conn_01x08 -> Connector_Generic:Conn_01x05
Connections:
- wire segments 12 -> 4
