File: circuit/9x9/9x9.sch (KiCad schematic (older format))
At the start: 172 parts, among them J1 Conn_01x06_Male, U1 ESP32-WROOM-32, U2 LD1117S33CTR

Commit message: v1.1
Parts:
- removed JOUT2: Conn_01x08_Shielded, Connector_JST:JST_SUR_BM08B-SURS-TF_1x08-1MP_P0.80mm_Vertical, symbol Connector_Generic:Conn_01x08
- added JOUT2: Conn_01x05, library:thick_header_01x05_3.3mm, symbol Connector_Generic:Conn_01x05
- J1: value Conn_01x06_Male -> Conn_01x10_Male; footprint Connector_PinHeader_2.54mm:PinHeader_2x03_P2.54mm_Vertical -> Connector_PinHeader_2.54mm:PinHeader_2x05_P2.54mm_Vertical; symbol Connector:Conn_01x06_Male -> Connector:Conn_01x10_Male
- JIN1, JOUT1: value Conn_01x08_Shielded -> Conn_01x05; footprint Connector_JST:JST_SUR_BM08B-SURS-TF_1x08-1MP_P0.80mm_Vertical -> library:thick_header_01x05_3.3mm; symbol Connector_Generic:Conn_01x08 -> Connector_Generic:Conn_01x05
Connections:
- wire segments 60 -> 66
Changed lines of the file:
@@
 EESchema Schematic File Version 4
-LIBS:tetris-cache
+LIBS:9x9-cache
 EELAYER 30 0
 EELAYER END
 $Descr A3 16535 11693
 encoding utf-8
-Sheet 2 3
+Sheet 1 1
 Title ""
 Date ""
@@
 	11200 3350 10400 3350
 $Comp
-L Connector:Conn_01x06_Male J1
+L Connector:Conn_01x10_Male J1
 U 1 1 5EF196AE
-P 11550 3450
-F 0 "J1" H 11522 3424 50  0000 R CNN
-F 1 "Conn_01x06_Male" H 11522 3333 50  0000 R CNN
-F 2 "Connector_PinHeader_2.54mm:PinHeader_2x03_P2.54mm_Vertical" H 11550 3450 50  0001 C CNN
-F 3 "~" H 11550 3450 50  0001 C CNN
-	1    11550 3450
+P 11550 3650
+F 0 "J1" H 11522 3624 50  0000 R CNN
+F 1 "Conn_01x10_Male" H 11522 3533 50  0000 R CNN
+F 2 "Connector_PinHeader_2.54mm:PinHeader_2x05_P2.54mm_Vertical" H 11550 3650 50  0001 C CNN
+F 3 "~" H 11550 3650 50  0001 C CNN
+	1    11550 3650
 	-1   0    0    -1
 $EndComp
@@
 L power:GND #PWR0347
 U 1 1 5EF360C7
-P 11350 3800
-F 0 "#PWR0347" H 11350 3550 50  0001 C CNN
-F 1 "GND" H 11355 3627 50  0000 C CNN
-F 2 "" H 11350 3800 50  0001 C CNN
-F 3 "" H 11350 3800 50  0001 C CNN
-	1    11350 3800
+P 11350 4200
+F 0 "#PWR0347" H 11350 3950 50  0001 C CNN
+F 1 "GND" H 11355 4027 50  0000 C CNN
+F 2 "" H 11350 4200 50  0001 C CNN
+F 3 "" H 11350 4200 50  0001 C CNN
+	1    11350 4200
 	1    0    0    -1
 $EndComp
-Wire Wire Line
-	11350 3750 11350 3800
 $Comp
 L power:+3.3V #PWR0348
@@
 OUT3
 $Comp
-L Connector_Generic:Conn_01x08 JIN1
-U 1 1 5EA2E46F
-P 7950 1100
-F 0 "JIN1" H 8030 1092 50  0000 L CNN
-F 1 "Conn_01x08_Shielded" H 8030 1001 50  0000 L CNN
-F 2 "Connector_JST:JST_SUR_BM08B-SURS-TF_1x08-1MP_P0.80mm_Vertical" H 7950 1100 50  0001 C CNN
-F 3 "~" H 7950 1100 50  0001 C CNN
-	1    7950 1100
-	1    0    0    -1
-$EndComp
-$Comp
-L Connector_Generic:Conn_01x08 JOUT1
+L Connector_Generic:Conn_01x05 JOUT1
 U 1 1 5EA3135F
 P 7950 2300
 F 0 "JOUT1" H 8030 2292 50  0000 L CNN
-F 1 "Conn_01x08_Shielded" H 8030 2201 50  0000 L CNN
-F 2 "Connector_JST:JST_SUR_BM08B-SURS-TF_1x08-1MP_P0.80mm_Vertical" H 7950 2300 50  0001 C CNN
+F 1 "Conn_01x05" H 8030 2201 50  0000 L CNN
+F 2 "library:thick_header_01x05_3.3mm" H 7950 2300 50  0001 C CNN
 F 3 "~" H 7950 2300 50  0001 C CNN
 	1    7950 2300
@@
 $EndComp
 $Comp
-L power:+5V #PWR0353
-U 1 1 5EA31D03
-P 7750 800
-F 0 "#PWR0353" H 7750 650 50  0001 C CNN
-F 1 "+5V" H 7765 973 50  0000 C CNN
-F 2 "" H 7750 800 50  0001 C CNN
-F 3 "" H 7750 800 50  0001 C CNN
-	1    7750 800
-	1    0    0    -1
-$EndComp
-Wire Wire Line
-	7750 900  7750 800
-Connection ~ 7750 800
-Wire Wire Line
-	7750 1400 7750 1500
-$Comp
 L power:GND #PWR0354
 U 1 1 5EA3B15A
-P 7750 1500
-F 0 "#PWR0354" H 7750 1250 50  0001 C CNN
-F 1 "GND" H 7755 1327 50  0000 C CNN
-F 2 "" H 7750 1500 50  0001 C CNN
-F 3 "" H 7750 1500 50  0001 C CNN
-	1    7750 1500
+P 7750 1300
+F 0 "#PWR0354" H 7750 1050 50  0001 C CNN
+F 1 "GND" H 7755 1127 50  0000 C CNN
+F 2 "" H 7750 1300 50  0001 C CNN
+F 3 "" H 7750 1300 50  0001 C CNN
+	1    7750 1300
 	1    0    0    -1
 $EndComp
-Connection ~ 7750 1500
-Wire Wire Line
-	7750 1300 7750 1400
-Connection ~ 7750 1400
-Text GLabel 7750 1000 0    50   Input ~ 0
+Text GLabel 7750 900  0    50   Input ~ 0
 IN1
-Text GLabel 7750 1100 0    50   Input ~ 0
+Text GLabel 7750 1000 0    50   Input ~ 0
 IN2
-Text GLabel 7750 1200 0    50   Input ~ 0
+Text GLabel 7750 1100 0    50   Input ~ 0
 IN3
-Wire Wire Line
-	7750 2100 7750 2000
-Wire Wire Line
-	7750 2500 7750 2600
-Connection ~ 7750 2600
-Wire Wire Line
-	7750 2600 7750 2700
 $Comp
 L power:GND #PWR0355
 U 1 1 5EA4CA66
-P 7750 2700
-F 0 "#PWR0355" H 7750 2450 50  0001 C CNN
-F 1 "GND" H 7755 2527 50  0000 C CNN
-F 2 "" H 7750 2700 50  0001 C CNN
-F 3 "" H 7750 2700 50  0001 C CNN
-	1    7750 2700
+P 7750 2500
+F 0 "#PWR0355" H 7750 2250 50  0001 C CNN
+F 1 "GND" H 7755 2327 50  0000 C CNN
+F 2 "" H 7750 2500 50  0001 C CNN
+F 3 "" H 7750 2500 50  0001 C CNN
+	1    7750 2500
 	1    0    0    -1
 $EndComp
-Connection ~ 7750 2700
 $Comp
 L power:+5V #PWR0356
 U 1 1 5EA4EDC8
-P 7750 2000
-F 0 "#PWR0356" H 7750 1850 50  0001 C CNN
-F 1 "+5V" H 7765 2173 50  0000 C CNN
-F 2 "" H 7750 2000 50  0001 C CNN
-F 3 "" H 7750 2000 50  0001 C CNN
-	1    7750 2000
+P 7350 2400
+F 0 "#PWR0356" H 7350 2250 50  0001 C CNN
+F 1 "+5V" H 7365 2573 50  0000 C CNN
+F 2 "" H 7350 2400 50  0001 C CNN
+F 3 "" H 7350 2400 50  0001 C CNN
+	1    7350 2400
 	1    0    0    -1
 $EndComp
-Connection ~ 7750 2000
-Text GLabel 7750 2200 0    50   Input ~ 0
+Text GLabel 7750 2100 0    50   Input ~ 0
 OUT1
-Text GLabel 7750 2300 0    50   Input ~ 0
+Text GLabel 7750 2200 0    50   Input ~ 0
 OUT2
-Text GLabel 7750 2400 0    50   Input ~ 0
+Text GLabel 7750 2300 0    50   Input ~ 0
 OUT3
-$Comp
-L Connector_Generic:Conn_01x08 JOUT2
-U 1 1 5EA589A7
-P 7950 3550
-F 0 "JOUT2" H 8030 3542 50  0000 L CNN
-F 1 "Conn_01x08_Shielded" H 8030 3451 50  0000 L CNN
-F 2 "Connector_JST:JST_SUR_BM08B-SURS-TF_1x08-1MP_P0.80mm_Vertical" H 7950 3550 50  0001 C CNN
-F 3 "~" H 7950 3550 50  0001 C CNN
-	1    7950 3550
-	1    0    0    -1
-$EndComp
 Wire Wire Line
-	7750 3350 7750 3250
+	11350 4200 11350 4150
+Wire Wire Line
+	10400 3850 10850 3850
+Wire Wire Line
+	10850 3850 10850 3750
+Wire Wire Line
+	10850 3750 11350 3750
+Wire Wire Line
+	10400 3950 10950 3950
+Wire Wire Line
+	10950 3950 10950 3850
+Wire Wire Line
+	10950 3850 11350 3850
 Wire Wire Line
-	7750 3750 7750 3850
-Connection ~ 7750 3850
+	10400 4050 11050 4050
 Wire Wire Line
-	7750 3850 7750 3950
+	11050 4050 11050 3950
+Wire Wire Line
+	11050 3950 11350 3950
+Wire Wire Line
+	10400 4150 11150 4150
+Wire Wire Line
+	11150 4150 11150 4050
+Wire Wire Line
+	11150 4050 11350 4050
+Wire Wire Line
+	7350 2400 7750 2400
+$Comp
+L Connector_Generic:Conn_01x05 JOUT2
+U 1 1 5EB06FC0
+P 7950 3150
+F 0 "JOUT2" H 8030 3142 50  0000 L CNN
+F 1 "Conn_01x05" H 8030 3051 50  0000 L CNN
+F 2 "library:thick_header_01x05_3.3mm" H 7950 3150 50  0001 C CNN
+F 3 "~" H 7950 3150 50  0001 C CNN
+	1    7950 3150
+	1    0    0    -1
+$EndComp
 $Comp
-L power:GND #PWR0357
-U 1 1 5EA589B1
-P 7750 3950
-F 0 "#PWR0357" H 7750 3700 50  0001 C CNN
-F 1 "GND" H 7755 3777 50  0000 C CNN
-F 2 "" H 7750 3950 50  0001 C CNN
-F 3 "" H 7750 3950 50  0001 C CNN
-	1    7750 3950
+L power:GND #PWR03
+U 1 1 5EB06FC6
+P 7750 3350
+F 0 "#PWR03" H 7750 3100 50  0001 C CNN
+F 1 "GND" H 7755 3177 50  0000 C CNN
+F 2 "" H 7750 3350 50  0001 C CNN
+F 3 "" H 7750 3350 50  0001 C CNN
+	1    7750 3350
 	1    0    0    -1
 $EndComp
-Connection ~ 7750 3950
 $Comp
-L power:+5V #PWR0358
-U 1 1 5EA589B8
-P 7750 3250
-F 0 "#PWR0358" H 7750 3100 50  0001 C CNN
-F 1 "+5V" H 7765 3423 50  0000 C CNN
-F 2 "" H 7750 3250 50  0001 C CNN
-F 3 "" H 7750 3250 50  0001 C CNN
-	1    7750 3250
+L power:+5V #PWR02
+U 1 1 5EB06FCC
+P 7350 3250
+F 0 "#PWR02" H 7350 3100 50  0001 C CNN
+F 1 "+5V" H 7365 3423 50  0000 C CNN
+F 2 "" H 7350 3250 50  0001 C CNN
+F 3 "" H 7350 3250 50  0001 C CNN
+	1    7350 3250
 	1    0    0    -1
 $EndComp
-Connection ~ 7750 3250
-Text GLabel 7750 3450 0    50   Input ~ 0
+Text GLabel 7750 2950 0    50   Input ~ 0
 OUT1
-Text GLabel 7750 3550 0    50   Input ~ 0
+Text GLabel 7750 3050 0    50   Input ~ 0
 OUT2
-Text GLabel 7750 3650 0    50   Input ~ 0
+Text GLabel 7750 3150 0    50   Input ~ 0
 OUT3
+Wire Wire Line
+	7350 3250 7750 3250
+$Comp
+L power:+5V #PWR01
+U 1 1 5EB092E0
+P 7350 1200
+F 0 "#PWR01" H 7350 1050 50  0001 C CNN
+F 1 "+5V" H 7365 1373 50  0000 C CNN
+F 2 "" H 7350 1200 50  0001 C CNN
+F 3 "" H 7350 1200 50  0001 C CNN
+	1    7350 1200
+	1    0    0    -1
+$EndComp
+Wire Wire Line
+	7350 1200 7750 1200
+$Comp
+L Connector_Generic:Conn_01x05 JIN1
+U 1 1 5EA2E46F
+P 7950 1100
+F 0 "JIN1" H 8030 1092 50  0000 L CNN
+F 1 "Conn_01x05" H 8030 1001 50  0000 L CNN
+F 2 "library:thick_header_01x05_3.3mm" H 7950 1100 50  0001 C CNN
+F 3 "~" H 7950 1100 50  0001 C CNN
+	1    7950 1100
+	1    0    0    -1
+$EndComp
 $EndSCHEMATC

Commit message: wip
Parts:
- added C85: 1800p, Capacitor_SMD:C_0805_2012Metric, symbol Device:C_Small
- added C86: 10u, Capacitor_SMD:C_0805_2012Metric, symbol Device:C_Small
- added C87: 68p, Capacitor_SMD:C_0805_2012Metric, symbol Device:C_Small
- added C88: 0.015u, Capacitor_SMD:C_0805_2012Metric, symbol Device:C_Small
- added C89: 0.1u, Capacitor_SMD:C_0805_2012Metric, symbol Device:C_Small
- added C90: 47u, Capacitor_SMD:C_0805_2012Metric, symbol Device:CP_Small
- added D82, D83: B240A, Diode_SMD:D_SMA_Handsoldering, symbol Device:D_Schottky
- added L1: 22u, Inductor_SMD:L_Vishay_IHLP-4040, symbol Device:L
- added R2: 21k, Resistor_SMD:R_0805_2012Metric, symbol Device:R_Small
- added R3: 10k, Resistor_SMD:R_0805_2012Metric, symbol Device:R_Small
- added R4: 1.91k, Resistor_SMD:R_0805_2012Metric, symbol Device:R_Small
- added U3: TPS54233, Package_SO:SOIC-8_3.9x4.9mm_P1.27mm, symbol Regulator_Switching:TPS54233
Connections:
- net +5V: now also D83.1 (K); no longer JIN1.4 (Pin_4), JOUT1.4 (Pin_4), JOUT2.4 (Pin_4)
- net GND: now also C86.2, C87.2, C88.2, C90.2, D82.2 (A), R2.2, R4.2, U3.7 (GND)
- new net: C89.2, U3.1 (BOOT)
- new net: C88.1, U3.4 (SS)
- new net: R3.2, R4.1, U3.5 (FB)
- new net: C85.1, C87.1, U3.6 (COMP)
- new net: C89.1, D82.1 (K), L1.1, U3.8 (PH)
- new net: C85.2, R2.1
- new net: C90.1, D83.2 (A), L1.2, R3.1
- new net +12V: C86.1, JIN1.4 (Pin_4), JOUT1.4 (Pin_4), JOUT2.4 (Pin_4), U3.2 (VIN)
